File: stm32f4discovery-daugherboard.brd (EAGLE design)
At the start: 100 x 71.1 mm, 41 parts

Commit message: small improvements
Parts:
- moved PWRDISCOVERY 2.65 mm to (84.6, 65.3)
Routing:
- net PWM_VIN: track 111.9 -> 134.8 mm
- net N$18: track 0.00 -> 17.9 mm
- net VIN: track 0.00 -> 16.5 mm, vias 0 -> 6
- net GND: track 137.1 -> 150.7 mm, vias 9 -> 15
- added copper zone on layer 1, net N$17
- added copper zone on layer 1, net N$19
- added copper zone on layer 1, net N$20
- added copper zone on layer 1, net N$21
- added copper zone on layer 1, net N$22
- added copper zone on layer 1, net N$23
- added copper zone on layer 1, net N$24
- added copper zone on layer 1, net N$25
- added copper zone on layer 1, net N$26
- added copper zone on layer 1, net N$27
