File: stm32f4discovery-daugherboard-v2.brd (EAGLE design)
At the start: 100 x 70 mm, 42 parts

Commit message: updated v2
Routing:
- net PC10: track 106.9 -> 163.8 mm
- net PC12: track 80.3 -> 136.5 mm
- net PC11: track 107.8 -> 163.4 mm
- net PE3: track 78.4 -> 125.9 mm
- net BOOT0: track 99.4 -> 124.8 mm
- net 3V: track 107.4 -> 132.1 mm
- net PWM_VIN: track 103.5 -> 84.0 mm
- net N$23: track 16.0 -> 0.00 mm
- net VIN: track 83.8 -> 71.1 mm, vias 24 -> 28
- net GND: track 8.13 -> 0.00 mm, vias 28 -> 24
- net PD5: track 52.9 -> 52.2 mm
- net PD6: track 51.6 -> 51.0 mm
- added copper zone on layer 1, net PWM_VIN
- removed copper zone on layer 1, net N$16

Commit message: sikscreen
sikscreen, paparazzi logo, prototyping are
Parts:
- added U$2, U$3: PAPARAZZI, paparazzi:PAPARAZZI
Routing:
- net PE6: track 86.0 -> 85.1 mm
- added copper zone on layer 1, net N$120
- added copper zone on layer 16, net N$121
- removed copper zone on layer 1, net N$13
Other:
- board text added: "5V"
- board text added: "ADC1"
- board text added: "ADC2"
- board text added: "ADC3"
- board text added: "ADC4"
- board text added: "ADC5"
- board text added: "ADC6"
- board text added: "Design by NeoFromMatrix (Marius Pfeffer)"
- board text added: "GND"
- board text added: "PPM IN"
- board text added: "PWM 0"
- board text added: "PWM 1"
- board text added: "PWM 10"
- board text added: "PWM 11"
- board text added: "PWM 2"
- board text added: "PWM 3"
- board text added: "PWM 4"
- board text added: "PWM 5"
- board text added: "PWM 6"
- board text added: "PWM 7"
- board text added: "PWM 8"
- board text added: "PWM 9"
- board text added: "PWM VIN"
- board text added: "Paparazzi"
- board text added: "RX"
- board text added: "SCL"
- board text added: "SDA"
- board text added: "SPEKTRUM BIND"
- board text added: "SPEKTRUM UART"
- board text added: "STM32F4 Discovery Daughterboard"
- board text added: "TODO: Sikscreen on both sides !"
- board text added: "TX"
- board text added: "The Free Autopilot"
- board text added: "VIN"
- board text added: "paparazziuav.org"
