File: stm32f4discovery-daugherboard-v2.sch (EAGLE design)
At the start: 42 parts

Commit message: sikscreen
sikscreen, paparazzi logo, prototyping are
Parts:
- added U$2, U$3: PAPARAZZI, paparazzi:PAPARAZZI
Other:
- note removed: "Add Open Source Hardware Logo !!!"
- note removed: "Add Paparazzi Penguin ! :)"
- moved on the sheet: BOOT0, BOOT1, C1, C2, C3, H5, H6, H7, H8, PWRDISCOVERY-1, PWRDISCOVERY-2, PWRDISCOVERY1-1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
