File: V1.0/stm32f4discovery_daughterboard.kicad_pcb (KiCad board)
At the start: 2 copper layers, 99.9 x 70 mm, 142 parts, among them P1 CONN_25X2, P2 CONN_25X2, T1 BC547

Commit message: added gerber
only first version, cleanup is required
Parts:
- moved R14 1.14 mm to (126.2, 123.7)
- moved T1 0.25 mm to (132.6, 119.1)
Routing:
- net 5V: track 14.5 -> 74.1 mm, vias 2 -> 6
- net (no net): track 35.0 -> 0.00 mm, vias 8 -> 0
- net PC8: track 12.5 -> 13.5 mm
